File: Hardware/PCB/harp rfid reader.kicad_sch (KiCad schematic)
At the start: 26 parts, among them IC1 FT232RL, IC2 NJM11100F1-TE2, J1 USB4105-GF-A, U2 TPD4E05U06DQA

Commit message: corrigidos erros em descrição de componentes
Parts:
- R12: Tolerance ±0.1% -> ±1%
- R17: Tolerance ±0.1% -> (none)
Changed lines of the file:
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@@
 			)
 		)
-		(property "Tolerance" "±0.1%"
+		(property "Tolerance" "±1%"
 			(at 142.24 121.92 0)
 			(hide yes)
@@
 			)
 		)
-		(property "Tolerance" "±0.1%"
+		(property "Tolerance" ""
 			(at 119.38 105.41 0)
 			(hide yes)
