File: Hardware/PCB/core.kicad_sch (KiCad schematic)
At the start: 36 parts, among them IC10 SN74LVC1G125DBVT, IC3 ATxmega32A4U-A, IC4 SN74LVC1G125DBVT, IC5 SN74LVC1G125DBVT, J2 282834-2, J3 NPPN051BFLD-RC, J4 NPPN071BFLC-RC, Q1 BC817-40W, Q2 NTF2955T1G, U1 ID-12/20SMD, X1 O 32,0-JT32C-A-K-3,3-LF

Commit message: MPN de IC4 IC5 IC10 não estavam correctos
. corrigidos MPN & footprints
. rerouting feito: DRC=0
. gerados ficheiros produção
Parts:
- IC10, IC4, IC5: value SN74LVC1G125DBVT -> MC74VHC1GT125DBVT1G; footprint Package_TO_SOT_SMD:SOT-23-5 -> Package_TO_SOT_SMD:SOT-353_SC-70-5; MPN SN74LVC1G125DBVT -> MC74VHC1GT125DBVT1G; OEPS Description IC: BUFFER NON-INVERT 1CH 3-STATE [SN74LVC1G125DBVT] [SOT-2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 -> IC: BUFFER NON-INVERT 1CH 3-STATE [MC74VHC1GT125DBVT1G] [SC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; OEPS PN OEPS080029 -> OEPS080169
Changed lines of the file:
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@@
 			)
 		)
-		(property "Value" "SN74LVC1G125DBVT"
+		(property "Value" "MC74VHC1GT125DBVT1G"
 			(at 187.452 152.146 0)
 			(show_name no)
@@
 			)
 		)
-		(property "Footprint" "Package_TO_SOT_SMD:SOT-23-5"
+		(property "Footprint" "Package_TO_SOT_SMD:SOT-353_SC-70-5"
 			(at 186.69 144.78 0)
 			(hide yes)
@@
 			)
 		)
-		(property "Description" "IC:   BUFFER NON-INVERT 1CH 3-STATE   [SN74LVC1G125DBVT] [SOT-23-5]"
+		(property "Description" "IC:   BUFFER NON-INVERT 1CH 3-STATE   [MC74VHC1GT125DBVT1G] [SC-74A]"
 			(at 186.69 144.78 0)
 			(hide yes)
@@
 			)
 		)
-		(property "MPN" "SN74LVC1G125DBVT"
+		(property "MPN" "MC74VHC1GT125DBVT1G"
 			(at 186.69 144.78 0)
 			(hide yes)
@@
 			)
 		)
-		(property "OEPS Description" "IC:   BUFFER NON-INVERT 1CH 3-STATE   [SN74LVC1G125DBVT] [SOT-23-5]"
+		(property "OEPS Description" "IC:   BUFFER NON-INVERT 1CH 3-STATE   [MC74VHC1GT125DBVT1G] [SC-74A]"
 			(at 186.69 144.78 0)
 			(hide yes)
@@
 			)
 		)
-		(property "OEPS PN" "OEPS080029"
+		(property "OEPS PN" "OEPS080169"
 			(at 186.69 144.78 0)
 			(hide yes)
@@
 			)
 		)
-		(property "Value" "SN74LVC1G125DBVT"
+		(property "Value" "MC74VHC1GT125DBVT1G"
 			(at 175.26 53.594 0)
 			(show_name no)
@@
 			)
 		)
-		(property "Footprint" "Package_TO_SOT_SMD:SOT-23-5"
+		(property "Footprint" "Package_TO_SOT_SMD:SOT-353_SC-70-5"
 			(at 175.26 45.72 0)
 			(hide yes)
@@
 			)
 		)
-		(property "Description" "IC:   BUFFER NON-INVERT 1CH 3-STATE   [SN74LVC1G125DBVT] [SOT-23-5]"
+		(property "Description" "IC:   BUFFER NON-INVERT 1CH 3-STATE   [MC74VHC1GT125DBVT1G] [SC-74A]"
 			(at 175.26 45.72 0)
 			(hide yes)
@@
 			)
 		)
-		(property "MPN" "SN74LVC1G125DBVT"
+		(property "MPN" "MC74VHC1GT125DBVT1G"
 			(at 175.26 45.72 0)
 			(hide yes)
@@
 			)
 		)
-		(property "OEPS Description" "IC:   BUFFER NON-INVERT 1CH 3-STATE   [SN74LVC1G125DBVT] [SOT-23-5]"
+		(property "OEPS Description" "IC:   BUFFER NON-INVERT 1CH 3-STATE   [MC74VHC1GT125DBVT1G] [SC-74A]"
 			(at 175.26 45.72 0)
 			(hide yes)
@@
 			)
 		)
-		(property "OEPS PN" "OEPS080029"
+		(property "OEPS PN" "OEPS080169"
 			(at 175.26 45.72 0)
 			(hide yes)
@@
 			)
 		)
-		(property "Value" "SN74LVC1G125DBVT"
+		(property "Value" "MC74VHC1GT125DBVT1G"
 			(at 177.8 98.298 0)
 			(show_name no)
@@
 			)
 		)
-		(property "Footprint" "Package_TO_SOT_SMD:SOT-23-5"
+		(property "Footprint" "Package_TO_SOT_SMD:SOT-353_SC-70-5"
 			(at 176.53 91.44 0)
 			(hide yes)
@@
 			)
 		)
-		(property "Description" "IC:   BUFFER NON-INVERT 1CH 3-STATE   [SN74LVC1G125DBVT] [SOT-23-5]"
+		(property "Description" "IC:   BUFFER NON-INVERT 1CH 3-STATE   [MC74VHC1GT125DBVT1G] [SC-74A]"
 			(at 176.53 91.44 0)
 			(hide yes)
@@
 			)
 		)
-		(property "MPN" "SN74LVC1G125DBVT"
+		(property "MPN" "MC74VHC1GT125DBVT1G"
 			(at 176.53 91.44 0)
 			(hide yes)
@@
 			)
 		)
-		(property "OEPS Description" "IC:   BUFFER NON-INVERT 1CH 3-STATE   [SN74LVC1G125DBVT] [SOT-23-5]"
+		(property "OEPS Description" "IC:   BUFFER NON-INVERT 1CH 3-STATE   [MC74VHC1GT125DBVT1G] [SC-74A]"
 			(at 176.53 91.44 0)
 			(hide yes)
@@
 			)
 		)
-		(property "OEPS PN" "OEPS080029"
+		(property "OEPS PN" "OEPS080169"
 			(at 176.53 91.44 0)
 			(hide yes)

Commit message: dorrecção em ligação módulo RFID
Connections:
- net +3V3: no longer J3.2 (Pin_2), U1.2 (RES)
- net VRFID: now also J3.2 (Pin_2), U1.2 (RES)
Changed lines of the file:
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@@
 	)
 	(junction
-		(at 262.89 57.15)
-		(diameter 0)
-		(color 0 0 0 0)
-	)
-	(junction
 		(at 86.36 25.4)
 		(diameter 0)
@@
 	)
 	(junction
+		(at 262.89 57.15)
+		(diameter 0)
+		(color 0 0 0 0)
+	)
+	(junction
 		(at 186.69 74.93)
 		(diameter 0)
@@
 	)
 	(junction
+		(at 262.89 48.26)
+		(diameter 0)
+		(color 0 0 0 0)
+	)
+	(junction
 		(at 160.02 45.72)
 		(diameter 0)
@@
 	(wire
 		(pts
+			(xy 262.89 48.26) (xy 262.89 46.99)
+		)
+		(stroke
+			(width 0.1524)
+			(type solid)
+		)
+	)
+	(wire
+		(pts
 			(xy 195.58 63.5) (xy 195.58 45.72)
 		)
@@
 	(wire
 		(pts
+			(xy 227.33 48.26) (xy 262.89 48.26)
+		)
+		(stroke
+			(width 0)
+			(type default)
+		)
+	)
+	(wire
+		(pts
 			(xy 148.59 149.86) (xy 148.59 144.78)
 		)
@@
 	(wire
 		(pts
-			(xy 227.33 64.77) (xy 227.33 58.42)
-		)
-		(stroke
-			(width 0)
-			(type default)
-		)
-	)
-	(wire
-		(pts
 			(xy 66.04 157.48) (xy 66.04 160.02)
 		)
@@
 	(wire
 		(pts
+			(xy 227.33 48.26) (xy 227.33 64.77)
+		)
+		(stroke
+			(width 0)
+			(type default)
+		)
+	)
+	(wire
+		(pts
 			(xy 264.16 69.85) (xy 265.43 69.85)
 		)
@@
 	(wire
 		(pts
-			(xy 262.89 57.15) (xy 262.89 50.8)
+			(xy 262.89 57.15) (xy 262.89 48.26)
 		)
 		(stroke
@@
 	)
 	(symbol
-		(lib_id "power:+5V")
-		(at 227.33 58.42 0)
-		(unit 1)
-		(body_style 1)
-		(exclude_from_sim no)
-		(in_bom yes)
-		(on_board yes)
-		(in_pos_files yes)
-		(dnp no)
-		(property "Reference" "#P+03"
-			(at 227.33 58.42 0)
-			(hide yes)
-			(show_name no)
-			(do_not_autoplace no)
-			(effects
-				(font
-					(size 1.27 1.27)
-				)
-			)
-		)
-		(property "Value" "+3V3"
-			(at 228.346 54.864 0)
-			(show_name no)
-			(do_not_autoplace no)
-			(effects
-				(font
-					(size 1.27 1.27)
-				)
-			)
-		)
-		(property "Footprint" ""
-			(at 227.33 58.42 0)
-			(hide yes)
-			(show_name no)
-			(do_not_autoplace no)
-			(effects
-				(font
-					(size 1.27 1.27)
-				)
-			)
-		)
-		(property "Datasheet" ""
-			(at 227.33 58.42 0)
-			(hide yes)
-			(show_name no)
-			(do_not_autoplace no)
-			(effects
-				(font
-					(size 1.27 1.27)
-				)
-			)
-		)
-		(property "Description" "Power symbol creates a global label with name \"+5V\""
-			(at 227.33 58.42 0)
-			(hide yes)
-			(show_name no)
-			(do_not_autoplace no)
-			(effects
-				(font
-					(size 1.27 1.27)
-				)
-			)
-		)
-		(pin "1"
-		)
-		(instances
-			(project "harp rfid reader"
-				(path "/d6d17c62-f9ae-4366-9aa9-0bf189dc20a6/e9956eac-47ad-4e7f-b529-fa68591fc6ae"
-					(reference "#P+03")
-					(unit 1)
-				)
-			)
-		)
-	)
-	(symbol
 		(lib_id "harp rfid reader-eagle-import:GND")
 		(at 181.61 104.14 0)
@@
 	(symbol
 		(lib_id "power:VDD")
-		(at 262.89 50.8 0)
+		(at 262.89 46.99 0)
 		(unit 1)
 		(body_style 1)
@@
 		(dnp no)
 		(property "Reference" "#PWR03"
-			(at 262.89 54.61 0)
+			(at 262.89 50.8 0)
 			(hide yes)
 			(show_name no)
@@
 		)
 		(property "Value" "VRFID"
-			(at 262.89 46.99 0)
+			(at 262.89 43.18 0)
 			(show_name no)
 			(do_not_autoplace no)
@@
 		)
 		(property "Footprint" ""
-			(at 262.89 50.8 0)
+			(at 262.89 46.99 0)
 			(hide yes)
 			(show_name no)
@@
 		)
 		(property "Datasheet" ""
-			(at 262.89 50.8 0)
+			(at 262.89 46.99 0)
 			(hide yes)
 			(show_name no)
@@
 		)
 		(property "Description" "Power symbol creates a global label with name \"VDD\""
-			(at 262.89 50.8 0)
+			(at 262.89 46.99 0)
 			(hide yes)
 			(show_name no)

Commit message: corrigidos erros em descrição de componentes
Parts:
- R14, R15: Tolerance ±0.1% -> (none)
Changed lines of the file:
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@@
 			)
 		)
-		(property "Tolerance" "±0.1%"
+		(property "Tolerance" ""
 			(at 168.91 109.22 0)
 			(hide yes)
@@
 			)
 		)
-		(property "Tolerance" "±0.1%"
+		(property "Tolerance" ""
 			(at 168.91 63.5 0)
 			(hide yes)
